File: kicad/tex.kicad_sch (KiCad schematic)
At the start: 173 parts, among them SW1 SW_Push, SW10 SW_Push, SW11 SW_Push, SW12 SW_Push, SW13 SW_Push, SW14 SW_Push, SW15 SW_Push, SW16 SW_Push, SW17 SW_Push, SW18 SW_Push, SW19 SW_Push, SW2 SW_Push, SW20 SW_Push, SW21 SW_Push, SW22 SW_Push, SW23 SW_Push, SW24 SW_Push, SW25 SW_Push, SW26 SW_Push, SW27 SW_Push, SW28 SW_Push, SW29 SW_Push, SW3 SW_Push, SW30 SW_Push, SW31 SW_Push, SW32 SW_Push, SW33 SW_Push, SW34 SW_Push, SW35 SW_Push, SW36 SW_Push, SW37 SW_Push, SW38 SW_Push, SW39 SW_Push, SW4 SW_Push, SW40 SW_Push, SW41 SW_Push, SW42 SW_Push, SW43 SW_Push, SW44 SW_Push, SW45 SW_Push, SW46 SW_Push, SW47 SW_Push, SW48 SW_Push, SW49 SW_Push, SW5 SW_Push, SW50 SW_Push, SW51 SW_Push, SW52 SW_Push, SW53 SW_Push, SW54 SW_Push, SW55 SW_Push, SW56 SW_Push, SW57 SW_Push, SW58 SW_Push, SW59 SW_Push, SW6 SW_Push, SW60 SW_Push, SW61 SW_Push, SW62 SW_Push, SW63 SW_Push, SW64 SW_Push, SW65 SW_Push, SW66 SW_Push, SW67 SW_Push, SW68 SW_Push, SW69 SW_Push, SW7 SW_Push, SW70 SW_Push, SW71 SW_Push, SW72 SW_Push, SW73 SW_Push, SW74 SW_Push, SW75 SW_Push, SW76 SW_Push, SW77 SW_Push, SW78 SW_Push, SW79 SW_Push, SW8 SW_Push, SW80 SW_Push, SW81 SW_Push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

Commit message: done
Parts:
- added J1: Testpoint, Connector_PinHeader_1.00mm:PinHeader_1x02_P1.00mm_Vertical, symbol Connector:Conn_01x02_Pin
- added L1, L10, L11, L12, L13, L14, L15, L16, L17, L18, L19, L2, L20, L21, L22, L23, L24, L25, L26, L27, L28, L29, L3, L30, L31, L32, L33, L34, L35, L36, L37, L38, L39, L4, L40, L41, L42, L43, L44, L45, L46, L47, L48, L49, L5, L50, L51, L52, L53, L54, L55, L56, L57, L58, L59, L6, L60, L61, L62, L63, L64, L65, L66, L67, L68, L69, L7, L70, L71, L72, L73, L74, L75, L76, L77, L78, L79, L8, L80, L81, L82, L83, L84, L9: WS2812B-2020, LED_SMD:LED_WS2812B-2020_PLCC4_2.0x2.0mm, symbol LED:WS2812B-2020
- added R3: 10k, Resistor_SMD:R_0603_1608Metric, symbol Device:R_Small
- added R4: 220 ohm, Resistor_SMD:R_0603_1608Metric, symbol Device:R_Small
Connections:
- net +5V: now also U2.5 (VCC), L1.4 (VDD), L10.4 (VDD), L11.4 (VDD), L12.4 (VDD), L13.4 (VDD), L14.4 (VDD), L15.4 (VDD), L16.4 (VDD), L17.4 (VDD), L18.4 (VDD), L19.4 (VDD), L2.4 (VDD), L20.4 (VDD), L21.4 (VDD), L22.4 (VDD), L23.4 (VDD), L24.4 (VDD), L25.4 (VDD), L26.4 (VDD), L27.4 (VDD), L28.4 (VDD), L29.4 (VDD), L3.4 (VDD), L30.4 (VDD), L31.4 (VDD), L32.4 (VDD), L33.4 (VDD), L34.4 (VDD), L35.4 (VDD), L36.4 (VDD), L37.4 (VDD), L38.4 (VDD), L39.4 (VDD), L4.4 (VDD), L40.4 (VDD), L41.4 (VDD), L42.4 (VDD), L43.4 (VDD), L44.4 (VDD), L45.4 (VDD), L46.4 (VDD), L47.4 (VDD), L48.4 (VDD), L49.4 (VDD), L5.4 (VDD), L50.4 (VDD), L51.4 (VDD), L52.4 (VDD), L53.4 (VDD), L54.4 (VDD), L55.4 (VDD), L56.4 (VDD), L57.4 (VDD), L58.4 (VDD), L59.4 (VDD), L6.4 (VDD), L60.4 (VDD), L61.4 (VDD), L62.4 (VDD), L63.4 (VDD), L64.4 (VDD), L65.4 (VDD), L66.4 (VDD), L67.4 (VDD), L68.4 (VDD), L69.4 (VDD), L7.4 (VDD), L70.4 (VDD), L71.4 (VDD), L72.4 (VDD), L73.4 (VDD), L74.4 (VDD), L75.4 (VDD), L76.4 (VDD), L77.4 (VDD), L78.4 (VDD), L79.4 (VDD), L8.4 (VDD), L80.4 (VDD), L81.4 (VDD), L82.4 (VDD), L83.4 (VDD), L84.4 (VDD), L9.4 (VDD)
- net C1: now also U1.5 (IO1)
- net C10: now also U1.15 (IO11)
- net C11: now also U1.16 (IO12)
- net C12: now also U1.17 (IO13)
- net C2: now also U1.6 (IO2)
- net C3: now also U1.8 (IO4)
- net C4: now also U1.9 (IO5)
- net C5: now also U1.10 (IO6)
- net C6: now also U1.11 (IO7)
- net C7: now also U1.12 (IO8)
- net C8: now also U1.13 (IO9)
- net C9: now also U1.14 (IO10)
- net GND: now also U1.1 (GND), U1.2 (GND), U1.42 (GND), U1.43 (GND), U1.46 (GND), U1.47 (GND), U1.48 (GND), U1.49 (GND), U1.50 (GND), U1.51 (GND), U1.52 (GND), U1.53 (GND), U1.54 (GND), U1.55 (GND), U1.56 (GND), U1.57 (GND), U1.58 (GND), U1.59 (GND), U1.60 (GND), U1.61 (GND), U1.62 (GND), U1.63 (GND), U1.64 (GND), U1.65 (GND), L1.2 (VSS), L10.2 (VSS), L11.2 (VSS), L12.2 (VSS), L13.2 (VSS), L14.2 (VSS), L15.2 (VSS), L16.2 (VSS), L17.2 (VSS), L18.2 (VSS), L19.2 (VSS), L2.2 (VSS), L20.2 (VSS), L21.2 (VSS), L22.2 (VSS), L23.2 (VSS), L24.2 (VSS), L25.2 (VSS), L26.2 (VSS), L27.2 (VSS), L28.2 (VSS), L29.2 (VSS), L3.2 (VSS), L30.2 (VSS), L31.2 (VSS), L32.2 (VSS), L33.2 (VSS), L34.2 (VSS), L35.2 (VSS), L36.2 (VSS), L37.2 (VSS), L38.2 (VSS), L39.2 (VSS), L4.2 (VSS), L40.2 (VSS), L41.2 (VSS), L42.2 (VSS), L43.2 (VSS), L44.2 (VSS), L45.2 (VSS), L46.2 (VSS), L47.2 (VSS), L48.2 (VSS), L49.2 (VSS), L5.2 (VSS), L50.2 (VSS), L51.2 (VSS), L52.2 (VSS), L53.2 (VSS), L54.2 (VSS), L55.2 (VSS), L56.2 (VSS), L57.2 (VSS), L58.2 (VSS), L59.2 (VSS), L6.2 (VSS), L60.2 (VSS), L61.2 (VSS), L62.2 (VSS), L63.2 (VSS), L64.2 (VSS), L65.2 (VSS), L66.2 (VSS), L67.2 (VSS), L68.2 (VSS), L69.2 (VSS), L7.2 (VSS), L70.2 (VSS), L71.2 (VSS), L72.2 (VSS), L73.2 (VSS), L74.2 (VSS), L75.2 (VSS), L76.2 (VSS), L77.2 (VSS), L78.2 (VSS), L79.2 (VSS), L8.2 (VSS), L80.2 (VSS), L81.2 (VSS), L82.2 (VSS), L83.2 (VSS), L84.2 (VSS), L9.2 (VSS), R3.2
- net R1: now also U1.18 (IO14)
- net R2: now also U1.19 (IO15)
- net R3: now also U1.20 (IO16)
- net R4: now also U1.21 (IO17)
- net R5: now also U1.22 (IO18)
- net R6: now also U1.25 (IO21)
- net R7: now also U1.30 (IO48)
- net GPIO42: now reaches U1.38 (IO42)
- net GPIO42: now also U2.2
- net at U1.4 (IO0): now also J1.1 (Pin_1)
- net at U2.4: now also R4.1
- new net: L14.1 (DOUT), L15.3 (DIN)
- new net: L13.1 (DOUT), L14.3 (DIN)
- new net: L69.1 (DOUT), L70.3 (DIN)
- new net: L68.1 (DOUT), L69.3 (DIN)
- new net: L10.3 (DIN), L9.1 (DOUT)
- new net: L8.1 (DOUT), L9.3 (DIN)
- new net: L56.1 (DOUT), L57.3 (DIN)
- new net: L55.1 (DOUT), L56.3 (DIN)
- new net: L3.1 (DOUT), L4.3 (DIN)
- new net: L2.1 (DOUT), L3.3 (DIN)
- new net: L67.1 (DOUT), L68.3 (DIN)
- new net: L66.1 (DOUT), L67.3 (DIN)
- new net: L38.1 (DOUT), L39.3 (DIN)
- new net: L37.1 (DOUT), L38.3 (DIN)
- new net: L49.1 (DOUT), L50.3 (DIN)
- new net: L10.1 (DOUT), L11.3 (DIN)
- new net: L41.1 (DOUT), L42.3 (DIN)
- new net: L40.1 (DOUT), L41.3 (DIN)
- new net: J1.2 (Pin_2), R3.1
- new net: L17.1 (DOUT), L18.3 (DIN)
- new net: L16.1 (DOUT), L17.3 (DIN)
- new net: L74.1 (DOUT), L75.3 (DIN)
- new net: L73.1 (DOUT), L74.3 (DIN)
- new net: L1.1 (DOUT), L2.3 (DIN)
- new net: L25.1 (DOUT), L26.3 (DIN)
- new net: L82.1 (DOUT), L83.3 (DIN)
- new net: L81.1 (DOUT), L82.3 (DIN)
- new net: L42.1 (DOUT), L43.3 (DIN)
- new net: L35.1 (DOUT), L36.3 (DIN)
- new net: L34.1 (DOUT), L35.3 (DIN)
- new net: L71.1 (DOUT), L72.3 (DIN)
- new net: L70.1 (DOUT), L71.3 (DIN)
- new net: L5.1 (DOUT), L6.3 (DIN)
- new net: L4.1 (DOUT), L5.3 (DIN)
- new net: L59.1 (DOUT), L60.3 (DIN)
- new net: L31.1 (DOUT), L32.3 (DIN)
- new net: L30.1 (DOUT), L31.3 (DIN)
- new net: L33.1 (DOUT), L34.3 (DIN)
- new net: L63.1 (DOUT), L64.3 (DIN)
- new net: L62.1 (DOUT), L63.3 (DIN)
- new net: L23.1 (DOUT), L24.3 (DIN)
- new net: L78.1 (DOUT), L79.3 (DIN)
- new net: L77.1 (DOUT), L78.3 (DIN)
- new net: L11.1 (DOUT), L12.3 (DIN)
- new net: L26.1 (DOUT), L27.3 (DIN)
- new net: L22.1 (DOUT), L23.3 (DIN)
- new net: L27.1 (DOUT), L28.3 (DIN)
- new net: L80.1 (DOUT), L81.3 (DIN)
- new net: L79.1 (DOUT), L80.3 (DIN)
- new net: L64.1 (DOUT), L65.3 (DIN)
- new net: L32.1 (DOUT), L33.3 (DIN)
- new net: L58.1 (DOUT), L59.3 (DIN)
- new net: L57.1 (DOUT), L58.3 (DIN)
- new net: L52.1 (DOUT), L53.3 (DIN)
- new net: L51.1 (DOUT), L52.3 (DIN)
- new net: L45.1 (DOUT), L46.3 (DIN)
- new net: L44.1 (DOUT), L45.3 (DIN)
- new net: L47.1 (DOUT), L48.3 (DIN)
- new net: L46.1 (DOUT), L47.3 (DIN)
- new net: L39.1 (DOUT), L40.3 (DIN)
- new net: L7.1 (DOUT), L8.3 (DIN)
- new net: L76.1 (DOUT), L77.3 (DIN)
- new net: L75.1 (DOUT), L76.3 (DIN)
- new net: L53.1 (DOUT), L54.3 (DIN)
- new net: L50.1 (DOUT), L51.3 (DIN)
- new net: L43.1 (DOUT), L44.3 (DIN)
- new net: L21.1 (DOUT), L22.3 (DIN)
- new net: L20.1 (DOUT), L21.3 (DIN)
- new net: L18.1 (DOUT), L19.3 (DIN)
- new net: L6.1 (DOUT), L7.3 (DIN)
- new net: L61.1 (DOUT), L62.3 (DIN)
- new net: L19.1 (DOUT), L20.3 (DIN)
- new net: L54.1 (DOUT), L55.3 (DIN)
- new net: L83.1 (DOUT), L84.3 (DIN)
- new net: L15.1 (DOUT), L16.3 (DIN)
- new net: L29.1 (DOUT), L30.3 (DIN)
- new net: L65.1 (DOUT), L66.3 (DIN)
- new net: L28.1 (DOUT), L29.3 (DIN)
- new net DIN: L1.3 (DIN), R4.2
- new net EOS1: L12.1 (DOUT), L13.3 (DIN)
- new net EOS2: L24.1 (DOUT), L25.3 (DIN)
- new net EOS3: L36.1 (DOUT), L37.3 (DIN)
- new net EOS4: L48.1 (DOUT), L49.3 (DIN)
- new net EOS5: L60.1 (DOUT), L61.3 (DIN)
- new net EOS6: L72.1 (DOUT), L73.3 (DIN)
- no-connect marks 8 -> 15
Other:
- moved on the sheet: R1, R2, U1, U2, USB1

Commit message: done
Parts:
- J1: footprint Connector_PinHeader_1.00mm:PinHeader_1x02_P1.00mm_Vertical -> Connector_PinSocket_2.00mm:PinSocket_1x02_P2.00mm_Vertical
Changed lines of the file:
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@@
 			)
 		)
-		(property "Footprint" "Connector_PinHeader_1.00mm:PinHeader_1x02_P1.00mm_Vertical"
+		(property "Footprint" "Connector_PinSocket_2.00mm:PinSocket_1x02_P2.00mm_Vertical"
 			(at 242.57 90.17 0)
 			(hide yes)
