File: kicad/tex.kicad_pcb (KiCad board)
At the start: 2 copper layers, 84 parts, among them SW1 SW_Push, SW10 SW_Push, SW11 SW_Push, SW12 SW_Push, SW13 SW_Push, SW14 SW_Push, SW15 SW_Push, SW16 SW_Push, SW17 SW_Push, SW18 SW_Push, SW19 SW_Push, SW2 SW_Push, SW20 SW_Push, SW21 SW_Push, SW22 SW_Push, SW23 SW_Push, SW24 SW_Push, SW25 SW_Push, SW26 SW_Push, SW27 SW_Push, SW28 SW_Push, SW29 SW_Push, SW3 SW_Push, SW30 SW_Push, SW31 SW_Push, SW32 SW_Push, SW33 SW_Push, SW34 SW_Push, SW35 SW_Push, SW36 SW_Push, SW37 SW_Push, SW38 SW_Push, SW39 SW_Push, SW4 SW_Push, SW40 SW_Push, SW41 SW_Push, SW42 SW_Push, SW43 SW_Push, SW44 SW_Push, SW45 SW_Push, SW46 SW_Push, SW47 SW_Push, SW48 SW_Push, SW49 SW_Push, SW5 SW_Push, SW50 SW_Push, SW51 SW_Push, SW52 SW_Push, SW53 SW_Push, SW54 SW_Push, SW55 SW_Push, SW56 SW_Push, SW57 SW_Push, SW58 SW_Push, SW59 SW_Push, SW6 SW_Push, SW60 SW_Push, SW61 SW_Push, SW62 SW_Push, SW63 SW_Push, SW64 SW_Push, SW65 SW_Push, SW66 SW_Push, SW67 SW_Push, SW68 SW_Push, SW69 SW_Push, SW7 SW_Push, SW70 SW_Push, SW71 SW_Push, SW72 SW_Push, SW73 SW_Push, SW74 SW_Push, SW75 SW_Push, SW76 SW_Push, SW77 SW_Push, SW78 SW_Push, SW79 SW_Push, SW8 SW_Push, SW80 SW_Push, SW81 SW_Push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

Commit message: done
Parts:
- added D1: 1N4148W, Diode_SMD:D_SOD-123, F.Cu at (1182.2, 419.3)
- added D10: 1N4148W, Diode_SMD:D_SOD-123, F.Cu at (1353.6, 419.3)
- added D11: 1N4148W, Diode_SMD:D_SOD-123, F.Cu at (1372.7, 419.3)
- added D12: 1N4148W, Diode_SMD:D_SOD-123, F.Cu at (1391.7, 419.3)
- added D13: 1N4148W, Diode_SMD:D_SOD-123, F.Cu at (1410.8, 419.3)
- added D14: 1N4148W, Diode_SMD:D_SOD-123, F.Cu at (1429.8, 419.3)
- added D15: 1N4148W, Diode_SMD:D_SOD-123, F.Cu at (1448.9, 419.3)
- added D16: 1N4148W, Diode_SMD:D_SOD-123, F.Cu at (1467.9, 419.3)
- added D17: 1N4148W, Diode_SMD:D_SOD-123, F.Cu at (1182.2, 438.4)
- added D18: 1N4148W, Diode_SMD:D_SOD-123, F.Cu at (1201.2, 438.4)
- added D19: 1N4148W, Diode_SMD:D_SOD-123, F.Cu at (1220.3, 438.4)
- added D2: 1N4148W, Diode_SMD:D_SOD-123, F.Cu at (1201.2, 419.3)
- added D20: 1N4148W, Diode_SMD:D_SOD-123, F.Cu at (1239.3, 438.4)
- added D21: 1N4148W, Diode_SMD:D_SOD-123, F.Cu at (1258.4, 438.4)
- added D22: 1N4148W, Diode_SMD:D_SOD-123, F.Cu at (1277.4, 438.4)
- added D23: 1N4148W, Diode_SMD:D_SOD-123, F.Cu at (1296.5, 438.4)
- added D24: 1N4148W, Diode_SMD:D_SOD-123, F.Cu at (1315.5, 438.4)
- added D25: 1N4148W, Diode_SMD:D_SOD-123, F.Cu at (1334.6, 438.4)
- added D26: 1N4148W, Diode_SMD:D_SOD-123, F.Cu at (1353.6, 438.4)
- added D27: 1N4148W, Diode_SMD:D_SOD-123, F.Cu at (1372.7, 438.4)
- added D28: 1N4148W, Diode_SMD:D_SOD-123, F.Cu at (1391.7, 438.4)
- added D29: 1N4148W, Diode_SMD:D_SOD-123, F.Cu at (1410.8, 438.4)
- added D3: 1N4148W, Diode_SMD:D_SOD-123, F.Cu at (1220.3, 419.3)
- added D30: 1N4148W, Diode_SMD:D_SOD-123, F.Cu at (1439.3, 438.4)
- added D31: 1N4148W, Diode_SMD:D_SOD-123, F.Cu at (1467.9, 438.4)
- added D32: 1N4148W, Diode_SMD:D_SOD-123, F.Cu at (1186.9, 457.4)
- added D33: 1N4148W, Diode_SMD:D_SOD-123, F.Cu at (1210.7, 457.4)
- added D34: 1N4148W, Diode_SMD:D_SOD-123, F.Cu at (1229.8, 457.4)
- added D35: 1N4148W, Diode_SMD:D_SOD-123, F.Cu at (1248.8, 457.4)
- added D36: 1N4148W, Diode_SMD:D_SOD-123, F.Cu at (1267.9, 457.4)
- added D37: 1N4148W, Diode_SMD:D_SOD-123, F.Cu at (1286.9, 457.4)
- added D38: 1N4148W, Diode_SMD:D_SOD-123, F.Cu at (1306.0, 457.4)
- added D39: 1N4148W, Diode_SMD:D_SOD-123, F.Cu at (1325.0, 457.4)
- added D4: 1N4148W, Diode_SMD:D_SOD-123, F.Cu at (1239.3, 419.3)
- added D40: 1N4148W, Diode_SMD:D_SOD-123, F.Cu at (1344.1, 457.4)
- added D41: 1N4148W, Diode_SMD:D_SOD-123, F.Cu at (1363.1, 457.4)
- added D42: 1N4148W, Diode_SMD:D_SOD-123, F.Cu at (1382.2, 457.4)
- added D43: 1N4148W, Diode_SMD:D_SOD-123, F.Cu at (1401.2, 457.4)
- added D44: 1N4148W, Diode_SMD:D_SOD-123, F.Cu at (1420.3, 457.4)
- added D45: 1N4148W, Diode_SMD:D_SOD-123, F.Cu at (1444.1, 457.4)
- added D46: 1N4148W, Diode_SMD:D_SOD-123, F.Cu at (1467.9, 457.4)
- added D47: 1N4148W, Diode_SMD:D_SOD-123, F.Cu at (1189.3, 476.5)
- added D48: 1N4148W, Diode_SMD:D_SOD-123, F.Cu at (1215.5, 476.5)
- added D49: 1N4148W, Diode_SMD:D_SOD-123, F.Cu at (1234.5, 476.5)
- added D5: 1N4148W, Diode_SMD:D_SOD-123, F.Cu at (1258.4, 419.3)
- added D50: 1N4148W, Diode_SMD:D_SOD-123, F.Cu at (1253.6, 476.5)
- added D51: 1N4148W, Diode_SMD:D_SOD-123, F.Cu at (1272.7, 476.5)
- added D52: 1N4148W, Diode_SMD:D_SOD-123, F.Cu at (1291.7, 476.5)
- added D53: 1N4148W, Diode_SMD:D_SOD-123, F.Cu at (1310.8, 476.5)
- added D54: 1N4148W, Diode_SMD:D_SOD-123, F.Cu at (1329.8, 476.5)
- added D55: 1N4148W, Diode_SMD:D_SOD-123, F.Cu at (1348.8, 476.5)
- added D56: 1N4148W, Diode_SMD:D_SOD-123, F.Cu at (1367.9, 476.5)
- added D57: 1N4148W, Diode_SMD:D_SOD-123, F.Cu at (1387.0, 476.5)
- added D58: 1N4148W, Diode_SMD:D_SOD-123, F.Cu at (1406.0, 476.5)
- added D59: 1N4148W, Diode_SMD:D_SOD-123, F.Cu at (1437.0, 476.5)
- added D6: 1N4148W, Diode_SMD:D_SOD-123, F.Cu at (1277.4, 419.3)
- added D60: 1N4148W, Diode_SMD:D_SOD-123, F.Cu at (1467.9, 476.5)
- added D61: 1N4148W, Diode_SMD:D_SOD-123, F.Cu at (1194.1, 495.5)
- added D62: 1N4148W, Diode_SMD:D_SOD-123, F.Cu at (1225.0, 495.5)
- added D63: 1N4148W, Diode_SMD:D_SOD-123, F.Cu at (1244.1, 495.5)
- added D64: 1N4148W, Diode_SMD:D_SOD-123, F.Cu at (1263.1, 495.5)
- added D65: 1N4148W, Diode_SMD:D_SOD-123, F.Cu at (1282.2, 495.5)
- added D66: 1N4148W, Diode_SMD:D_SOD-123, F.Cu at (1301.2, 495.5)
- added D67: 1N4148W, Diode_SMD:D_SOD-123, F.Cu at (1320.3, 495.5)
- added D68: 1N4148W, Diode_SMD:D_SOD-123, F.Cu at (1339.3, 495.5)
- added D69: 1N4148W, Diode_SMD:D_SOD-123, F.Cu at (1358.4, 495.5)
- added D7: 1N4148W, Diode_SMD:D_SOD-123, F.Cu at (1296.5, 419.3)
- added D70: 1N4148W, Diode_SMD:D_SOD-123, F.Cu at (1377.4, 495.5)
- added D71: 1N4148W, Diode_SMD:D_SOD-123, F.Cu at (1396.5, 495.5)
- added D72: 1N4148W, Diode_SMD:D_SOD-123, F.Cu at (1422.7, 495.5)
- added D73: 1N4148W, Diode_SMD:D_SOD-123, F.Cu at (1448.9, 495.5)
- added D74: 1N4148W, Diode_SMD:D_SOD-123, F.Cu at (1467.9, 495.5)
- added D75: 1N4148W, Diode_SMD:D_SOD-123, F.Cu at (1184.5, 514.6)
- added D76: 1N4148W, Diode_SMD:D_SOD-123, F.Cu at (1208.4, 514.6)
- added D77: 1N4148W, Diode_SMD:D_SOD-123, F.Cu at (1232.2, 514.6)
- added D78: 1N4148W, Diode_SMD:D_SOD-123, F.Cu at (1303.6, 514.6)
- added D79: 1N4148W, Diode_SMD:D_SOD-123, F.Cu at (1372.7, 514.6)
- added D8: 1N4148W, Diode_SMD:D_SOD-123, F.Cu at (1315.5, 419.3)
- added D80: 1N4148W, Diode_SMD:D_SOD-123, F.Cu at (1391.7, 514.6)
- added D81: 1N4148W, Diode_SMD:D_SOD-123, F.Cu at (1410.8, 514.6)
- added D82: 1N4148W, Diode_SMD:D_SOD-123, F.Cu at (1429.8, 514.6)
- added D83: 1N4148W, Diode_SMD:D_SOD-123, F.Cu at (1448.9, 514.6)
- added D84: 1N4148W, Diode_SMD:D_SOD-123, F.Cu at (1467.9, 514.6)
- added D9: 1N4148W, Diode_SMD:D_SOD-123, F.Cu at (1334.6, 419.3)
- added L1: WS2812B-2020, LED_SMD:LED_WS2812B-2020_PLCC4_2.0x2.0mm, F.Cu at (1182.2, 412.3)
- added L10: WS2812B-2020, LED_SMD:LED_WS2812B-2020_PLCC4_2.0x2.0mm, F.Cu at (1353.6, 412.3)
- added L11: WS2812B-2020, LED_SMD:LED_WS2812B-2020_PLCC4_2.0x2.0mm, F.Cu at (1372.7, 412.3)
- added L12: WS2812B-2020, LED_SMD:LED_WS2812B-2020_PLCC4_2.0x2.0mm, F.Cu at (1391.7, 412.3)
- added L13: WS2812B-2020, LED_SMD:LED_WS2812B-2020_PLCC4_2.0x2.0mm, F.Cu at (1410.8, 412.3)
- added L14: WS2812B-2020, LED_SMD:LED_WS2812B-2020_PLCC4_2.0x2.0mm, F.Cu at (1429.8, 412.3)
- added L15: WS2812B-2020, LED_SMD:LED_WS2812B-2020_PLCC4_2.0x2.0mm, F.Cu at (1448.9, 412.3)
- added L16: WS2812B-2020, LED_SMD:LED_WS2812B-2020_PLCC4_2.0x2.0mm, F.Cu at (1467.9, 412.3)
- added L17: WS2812B-2020, LED_SMD:LED_WS2812B-2020_PLCC4_2.0x2.0mm, F.Cu at (1182.2, 431.4)
- added L18: WS2812B-2020, LED_SMD:LED_WS2812B-2020_PLCC4_2.0x2.0mm, F.Cu at (1201.2, 431.4)
- added L19: WS2812B-2020, LED_SMD:LED_WS2812B-2020_PLCC4_2.0x2.0mm, F.Cu at (1220.3, 431.4)
- added L2: WS2812B-2020, LED_SMD:LED_WS2812B-2020_PLCC4_2.0x2.0mm, F.Cu at (1201.2, 412.3)
- added L20: WS2812B-2020, LED_SMD:LED_WS2812B-2020_PLCC4_2.0x2.0mm, F.Cu at (1239.3, 431.4)
- added L21: WS2812B-2020, LED_SMD:LED_WS2812B-2020_PLCC4_2.0x2.0mm, F.Cu at (1258.4, 431.4)
- added L22: WS2812B-2020, LED_SMD:LED_WS2812B-2020_PLCC4_2.0x2.0mm, F.Cu at (1277.4, 431.4)
- added L23: WS2812B-2020, LED_SMD:LED_WS2812B-2020_PLCC4_2.0x2.0mm, F.Cu at (1296.5, 431.4)
- added L24: WS2812B-2020, LED_SMD:LED_WS2812B-2020_PLCC4_2.0x2.0mm, F.Cu at (1315.5, 431.4)
- added L25: WS2812B-2020, LED_SMD:LED_WS2812B-2020_PLCC4_2.0x2.0mm, F.Cu at (1334.6, 431.4)
- added L26: WS2812B-2020, LED_SMD:LED_WS2812B-2020_PLCC4_2.0x2.0mm, F.Cu at (1353.6, 431.4)
- added L27: WS2812B-2020, LED_SMD:LED_WS2812B-2020_PLCC4_2.0x2.0mm, F.Cu at (1372.7, 431.4)
- added L28: WS2812B-2020, LED_SMD:LED_WS2812B-2020_PLCC4_2.0x2.0mm, F.Cu at (1391.7, 431.4)
- added L29: WS2812B-2020, LED_SMD:LED_WS2812B-2020_PLCC4_2.0x2.0mm, F.Cu at (1410.8, 431.4)
- added L3: WS2812B-2020, LED_SMD:LED_WS2812B-2020_PLCC4_2.0x2.0mm, F.Cu at (1220.3, 412.3)
- added L30: WS2812B-2020, LED_SMD:LED_WS2812B-2020_PLCC4_2.0x2.0mm, F.Cu at (1439.3, 431.4)
- added L31: WS2812B-2020, LED_SMD:LED_WS2812B-2020_PLCC4_2.0x2.0mm, F.Cu at (1467.9, 431.4)
- added L32: WS2812B-2020, LED_SMD:LED_WS2812B-2020_PLCC4_2.0x2.0mm, F.Cu at (1186.9, 450.4)
- added L33: WS2812B-2020, LED_SMD:LED_WS2812B-2020_PLCC4_2.0x2.0mm, F.Cu at (1210.7, 450.4)
- added L34: WS2812B-2020, LED_SMD:LED_WS2812B-2020_PLCC4_2.0x2.0mm, F.Cu at (1229.8, 450.4)
- added L35: WS2812B-2020, LED_SMD:LED_WS2812B-2020_PLCC4_2.0x2.0mm, F.Cu at (1248.8, 450.4)
- added L36: WS2812B-2020, LED_SMD:LED_WS2812B-2020_PLCC4_2.0x2.0mm, F.Cu at (1267.9, 450.4)
- added L37: WS2812B-2020, LED_SMD:LED_WS2812B-2020_PLCC4_2.0x2.0mm, F.Cu at (1286.9, 450.4)
- added L38: WS2812B-2020, LED_SMD:LED_WS2812B-2020_PLCC4_2.0x2.0mm, F.Cu at (1306.0, 450.4)
- added L39: WS2812B-2020, LED_SMD:LED_WS2812B-2020_PLCC4_2.0x2.0mm, F.Cu at (1325.0, 450.4)
- added L4: WS2812B-2020, LED_SMD:LED_WS2812B-2020_PLCC4_2.0x2.0mm, F.Cu at (1239.3, 412.3)
- added L40: WS2812B-2020, LED_SMD:LED_WS2812B-2020_PLCC4_2.0x2.0mm, F.Cu at (1344.1, 450.4)
- added L41: WS2812B-2020, LED_SMD:LED_WS2812B-2020_PLCC4_2.0x2.0mm, F.Cu at (1363.1, 450.4)
- added L42: WS2812B-2020, LED_SMD:LED_WS2812B-2020_PLCC4_2.0x2.0mm, F.Cu at (1382.2, 450.4)
- added L43: WS2812B-2020, LED_SMD:LED_WS2812B-2020_PLCC4_2.0x2.0mm, F.Cu at (1401.2, 450.4)
- added L44: WS2812B-2020, LED_SMD:LED_WS2812B-2020_PLCC4_2.0x2.0mm, F.Cu at (1420.3, 450.4)
- added L45: WS2812B-2020, LED_SMD:LED_WS2812B-2020_PLCC4_2.0x2.0mm, F.Cu at (1444.1, 450.4)
- added L46: WS2812B-2020, LED_SMD:LED_WS2812B-2020_PLCC4_2.0x2.0mm, F.Cu at (1467.9, 450.4)
- added L47: WS2812B-2020, LED_SMD:LED_WS2812B-2020_PLCC4_2.0x2.0mm, F.Cu at (1189.3, 469.5)
- added L48: WS2812B-2020, LED_SMD:LED_WS2812B-2020_PLCC4_2.0x2.0mm, F.Cu at (1215.5, 469.5)
- added L49: WS2812B-2020, LED_SMD:LED_WS2812B-2020_PLCC4_2.0x2.0mm, F.Cu at (1234.5, 469.5)
- added L5: WS2812B-2020, LED_SMD:LED_WS2812B-2020_PLCC4_2.0x2.0mm, F.Cu at (1258.4, 412.3)
- added L50: WS2812B-2020, LED_SMD:LED_WS2812B-2020_PLCC4_2.0x2.0mm, F.Cu at (1253.6, 469.5)
- added L51: WS2812B-2020, LED_SMD:LED_WS2812B-2020_PLCC4_2.0x2.0mm, F.Cu at (1272.7, 469.5)
- added L52: WS2812B-2020, LED_SMD:LED_WS2812B-2020_PLCC4_2.0x2.0mm, F.Cu at (1291.7, 469.5)
- added L53: WS2812B-2020, LED_SMD:LED_WS2812B-2020_PLCC4_2.0x2.0mm, F.Cu at (1310.8, 469.5)
- added L54: WS2812B-2020, LED_SMD:LED_WS2812B-2020_PLCC4_2.0x2.0mm, F.Cu at (1329.8, 469.5)
- added L55: WS2812B-2020, LED_SMD:LED_WS2812B-2020_PLCC4_2.0x2.0mm, F.Cu at (1348.8, 469.5)
- added L56: WS2812B-2020, LED_SMD:LED_WS2812B-2020_PLCC4_2.0x2.0mm, F.Cu at (1367.9, 469.5)
- added L57: WS2812B-2020, LED_SMD:LED_WS2812B-2020_PLCC4_2.0x2.0mm, F.Cu at (1387.0, 469.5)
- added L58: WS2812B-2020, LED_SMD:LED_WS2812B-2020_PLCC4_2.0x2.0mm, F.Cu at (1406.0, 469.5)
- added L59: WS2812B-2020, LED_SMD:LED_WS2812B-2020_PLCC4_2.0x2.0mm, F.Cu at (1437.0, 469.5)
- added L6: WS2812B-2020, LED_SMD:LED_WS2812B-2020_PLCC4_2.0x2.0mm, F.Cu at (1277.4, 412.3)
- added L60: WS2812B-2020, LED_SMD:LED_WS2812B-2020_PLCC4_2.0x2.0mm, F.Cu at (1467.9, 469.5)
- added L61: WS2812B-2020, LED_SMD:LED_WS2812B-2020_PLCC4_2.0x2.0mm, F.Cu at (1194.1, 488.5)
- added L62: WS2812B-2020, LED_SMD:LED_WS2812B-2020_PLCC4_2.0x2.0mm, F.Cu at (1225.0, 488.5)
- added L63: WS2812B-2020, LED_SMD:LED_WS2812B-2020_PLCC4_2.0x2.0mm, F.Cu at (1244.1, 488.5)
- added L64: WS2812B-2020, LED_SMD:LED_WS2812B-2020_PLCC4_2.0x2.0mm, F.Cu at (1263.1, 488.5)
- added L65: WS2812B-2020, LED_SMD:LED_WS2812B-2020_PLCC4_2.0x2.0mm, F.Cu at (1282.2, 488.5)
- added L66: WS2812B-2020, LED_SMD:LED_WS2812B-2020_PLCC4_2.0x2.0mm, F.Cu at (1301.2, 488.5)
- added L67: WS2812B-2020, LED_SMD:LED_WS2812B-2020_PLCC4_2.0x2.0mm, F.Cu at (1320.3, 488.5)
- added L68: WS2812B-2020, LED_SMD:LED_WS2812B-2020_PLCC4_2.0x2.0mm, F.Cu at (1339.3, 488.5)
- added L69: WS2812B-2020, LED_SMD:LED_WS2812B-2020_PLCC4_2.0x2.0mm, F.Cu at (1358.4, 488.5)
- added L7: WS2812B-2020, LED_SMD:LED_WS2812B-2020_PLCC4_2.0x2.0mm, F.Cu at (1296.5, 412.3)
- added L70: WS2812B-2020, LED_SMD:LED_WS2812B-2020_PLCC4_2.0x2.0mm, F.Cu at (1377.4, 488.5)
- added L71: WS2812B-2020, LED_SMD:LED_WS2812B-2020_PLCC4_2.0x2.0mm, F.Cu at (1396.5, 488.5)
- added L72: WS2812B-2020, LED_SMD:LED_WS2812B-2020_PLCC4_2.0x2.0mm, F.Cu at (1422.7, 488.5)
- added L73: WS2812B-2020, LED_SMD:LED_WS2812B-2020_PLCC4_2.0x2.0mm, F.Cu at (1448.9, 488.5)
- added L74: WS2812B-2020, LED_SMD:LED_WS2812B-2020_PLCC4_2.0x2.0mm, F.Cu at (1467.9, 488.5)
- added L75: WS2812B-2020, LED_SMD:LED_WS2812B-2020_PLCC4_2.0x2.0mm, F.Cu at (1184.5, 507.6)
- added L76: WS2812B-2020, LED_SMD:LED_WS2812B-2020_PLCC4_2.0x2.0mm, F.Cu at (1208.4, 507.6)
- added L77: WS2812B-2020, LED_SMD:LED_WS2812B-2020_PLCC4_2.0x2.0mm, F.Cu at (1232.2, 507.6)
- added L78: WS2812B-2020, LED_SMD:LED_WS2812B-2020_PLCC4_2.0x2.0mm, F.Cu at (1303.6, 507.6)
- added L79: WS2812B-2020, LED_SMD:LED_WS2812B-2020_PLCC4_2.0x2.0mm, F.Cu at (1372.7, 507.6)
- added L8: WS2812B-2020, LED_SMD:LED_WS2812B-2020_PLCC4_2.0x2.0mm, F.Cu at (1315.5, 412.3)
- added L80: WS2812B-2020, LED_SMD:LED_WS2812B-2020_PLCC4_2.0x2.0mm, F.Cu at (1391.7, 507.6)
- added L81: WS2812B-2020, LED_SMD:LED_WS2812B-2020_PLCC4_2.0x2.0mm, F.Cu at (1410.8, 507.6)
- added L82: WS2812B-2020, LED_SMD:LED_WS2812B-2020_PLCC4_2.0x2.0mm, F.Cu at (1429.8, 507.6)
- added L83: WS2812B-2020, LED_SMD:LED_WS2812B-2020_PLCC4_2.0x2.0mm, F.Cu at (1448.9, 507.6)
- added L84: WS2812B-2020, LED_SMD:LED_WS2812B-2020_PLCC4_2.0x2.0mm, F.Cu at (1467.9, 507.6)
- added L9: WS2812B-2020, LED_SMD:LED_WS2812B-2020_PLCC4_2.0x2.0mm, F.Cu at (1334.6, 412.3)
- added R1: 5.1k, Resistor_SMD:R_0603_1608Metric, B.Cu at (1316.6, 508.1)
- added R2: 5.1k, Resistor_SMD:R_0603_1608Metric, B.Cu at (1316.6, 510.6)
- added U1: ESP32-S3-MINI-1, RF_Module:ESP32-S2-MINI-1, B.Cu at (1340.2, 513.9)
- added U2: 74AHCT1G125, Package_TO_SOT_SMD:SOT-353_SC-70-5, B.Cu at (1165.5, 408.0)
- added USB1: USB-C, easyeda2kicad:USB-C-SMD_TYPE-C-31-M-31, B.Cu at (1323.9, 510.3)
- SW1, SW10, SW11, SW12, SW13, SW14, SW15, SW16, SW17, SW18, SW19, SW2, SW20, SW21, SW22, SW23, SW24, SW25, SW26, SW27, SW28, SW29, SW3, SW30, SW31, SW32, SW33, SW34, SW35, SW36, SW37, SW38, SW39, SW4, SW40, SW41, SW42, SW43, SW44, SW45, SW46, SW47, SW48, SW49, SW5, SW50, SW51, SW52, SW53, SW54, SW55, SW56, SW57, SW58, SW59, SW6, SW60, SW61, SW62, SW63, SW64, SW65, SW66, SW67, SW68, SW69, SW7, SW70, SW71, SW72, SW73, SW74, SW75, SW76, SW77, SW78, SW79, SW8, SW80, SW81, SW82, SW83, SW84, SW9: footprint Button_Switch_Keyboard:SW_Cherry_MX_1.00u_Plate -> Button_Switch_Keyboard:SW_Cherry_MX_1.00u_PCB
- moved SW32 671.7 mm to (1179.9, 447.4)
- moved SW75 669.9 mm to (1177.5, 504.6)
- moved SW33 666.6 mm to (1203.7, 447.4)
- moved SW76 660.9 mm to (1201.4, 504.6)
- moved SW77 653.0 mm to (1225.2, 504.6)
- moved SW17 635.1 mm to (1175.2, 428.4)
- moved SW61 634.4 mm to (1187.1, 485.5)
- moved SW18 632.4 mm to (1194.2, 428.4)
- moved SW22 631.1 mm to (1270.4, 428.4)
- moved SW19 630.7 mm to (1213.3, 428.4)
- moved SW21 630.0 mm to (1251.4, 428.4)
- moved SW20 629.9 mm to (1232.3, 428.4)
- moved SW62 619.7 mm to (1218.0, 485.5)
- moved SW63 615.4 mm to (1237.1, 485.5)
- moved SW64 612.1 mm to (1256.1, 485.5)
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Connections:
- SW1 pad 1: unconnected-(SW1-Pad1) -> Net-(D1-A)
- SW1 pad 2: unconnected-(SW1-Pad2) -> /R1
- SW10 pad 1: unconnected-(SW10-Pad1) -> Net-(D10-A)
- SW10 pad 2: unconnected-(SW10-Pad2) -> /R1
- SW11 pad 1: unconnected-(SW11-Pad1) -> Net-(D11-A)
- SW11 pad 2: unconnected-(SW11-Pad2) -> /R1
- SW12 pad 1: unconnected-(SW12-Pad1) -> Net-(D12-A)
- SW12 pad 2: unconnected-(SW12-Pad2) -> /R1
- SW13 pad 1: unconnected-(SW13-Pad1) -> Net-(D1-K)
- SW13 pad 2: unconnected-(SW13-Pad2) -> /R2
- SW14 pad 1: unconnected-(SW14-Pad1) -> Net-(D14-A)
- SW14 pad 2: unconnected-(SW14-Pad2) -> /R2
- SW15 pad 1: unconnected-(SW15-Pad1) -> Net-(D15-A)
- SW15 pad 2: unconnected-(SW15-Pad2) -> /R2
- SW16 pad 1: unconnected-(SW16-Pad1) -> Net-(D16-A)
- SW16 pad 2: unconnected-(SW16-Pad2) -> /R2
- SW17 pad 1: unconnected-(SW17-Pad1) -> Net-(D17-A)
- SW17 pad 2: unconnected-(SW17-Pad2) -> /R2
- SW18 pad 1: unconnected-(SW18-Pad1) -> Net-(D18-A)
- SW18 pad 2: unconnected-(SW18-Pad2) -> /R2
- SW19 pad 1: unconnected-(SW19-Pad1) -> Net-(D19-A)
- SW19 pad 2: unconnected-(SW19-Pad2) -> /R2
- SW2 pad 1: unconnected-(SW2-Pad1) -> Net-(D2-A)
- SW2 pad 2: unconnected-(SW2-Pad2) -> /R1
- SW20 pad 1: unconnected-(SW20-Pad1) -> Net-(D20-A)
- SW20 pad 2: unconnected-(SW20-Pad2) -> /R2
- SW21 pad 1: unconnected-(SW21-Pad1) -> Net-(D21-A)
- SW21 pad 2: unconnected-(SW21-Pad2) -> /R2
- SW22 pad 1: unconnected-(SW22-Pad1) -> Net-(D10-K)
- SW22 pad 2: unconnected-(SW22-Pad2) -> /R2
- SW23 pad 1: unconnected-(SW23-Pad1) -> Net-(D11-K)
- SW23 pad 2: unconnected-(SW23-Pad2) -> /R2
- SW24 pad 1: unconnected-(SW24-Pad1) -> Net-(D12-K)
- SW24 pad 2: unconnected-(SW24-Pad2) -> /R2
- SW25 pad 1: unconnected-(SW25-Pad1) -> Net-(D13-K)
- SW25 pad 2: unconnected-(SW25-Pad2) -> /R3
- SW26 pad 1: unconnected-(SW26-Pad1) -> Net-(D14-K)
- SW26 pad 2: unconnected-(SW26-Pad2) -> /R3
- SW27 pad 1: unconnected-(SW27-Pad1) -> Net-(D15-K)
- SW27 pad 2: unconnected-(SW27-Pad2) -> /R3
- SW28 pad 1: unconnected-(SW28-Pad1) -> Net-(D16-K)
- SW28 pad 2: unconnected-(SW28-Pad2) -> /R3
- SW29 pad 1: unconnected-(SW29-Pad1) -> Net-(D17-K)
- SW29 pad 2: unconnected-(SW29-Pad2) -> /R3
- SW3 pad 1: unconnected-(SW3-Pad1) -> Net-(D3-A)
- SW3 pad 2: unconnected-(SW3-Pad2) -> /R1
- SW30 pad 1: unconnected-(SW30-Pad1) -> Net-(D18-K)
- SW30 pad 2: unconnected-(SW30-Pad2) -> /R3
- SW31 pad 1: unconnected-(SW31-Pad1) -> Net-(D19-K)
- SW31 pad 2: unconnected-(SW31-Pad2) -> /R3
- SW32 pad 1: unconnected-(SW32-Pad1) -> Net-(D20-K)
- SW32 pad 2: unconnected-(SW32-Pad2) -> /R3
- SW33 pad 1: unconnected-(SW33-Pad1) -> Net-(D21-K)
- SW33 pad 2: unconnected-(SW33-Pad2) -> /R3
- SW34 pad 1: unconnected-(SW34-Pad1) -> Net-(D22-K)
- SW34 pad 2: unconnected-(SW34-Pad2) -> /R3
- SW35 pad 1: unconnected-(SW35-Pad1) -> Net-(D23-K)
- SW35 pad 2: unconnected-(SW35-Pad2) -> /R3
- SW36 pad 1: unconnected-(SW36-Pad1) -> Net-(D24-K)
- SW36 pad 2: unconnected-(SW36-Pad2) -> /R3
- SW37 pad 1: unconnected-(SW37-Pad1) -> Net-(D25-K)
- SW37 pad 2: unconnected-(SW37-Pad2) -> /R4
- SW38 pad 1: unconnected-(SW38-Pad1) -> Net-(D26-K)
- SW38 pad 2: unconnected-(SW38-Pad2) -> /R4
- SW39 pad 1: unconnected-(SW39-Pad1) -> Net-(D27-K)
- SW39 pad 2: unconnected-(SW39-Pad2) -> /R4
- SW4 pad 1: unconnected-(SW4-Pad1) -> Net-(D4-A)
- SW4 pad 2: unconnected-(SW4-Pad2) -> /R1
- SW40 pad 1: unconnected-(SW40-Pad1) -> Net-(D28-K)
- SW40 pad 2: unconnected-(SW40-Pad2) -> /R4
- SW41 pad 1: unconnected-(SW41-Pad1) -> Net-(D29-K)
- SW41 pad 2: unconnected-(SW41-Pad2) -> /R4
- SW42 pad 1: unconnected-(SW42-Pad1) -> Net-(D30-K)
- SW42 pad 2: unconnected-(SW42-Pad2) -> /R4
- SW43 pad 1: unconnected-(SW43-Pad1) -> Net-(D31-K)
- SW43 pad 2: unconnected-(SW43-Pad2) -> /R4
- SW44 pad 1: unconnected-(SW44-Pad1) -> Net-(D32-K)
- SW44 pad 2: unconnected-(SW44-Pad2) -> /R4
- SW45 pad 1: unconnected-(SW45-Pad1) -> Net-(D33-K)
- SW45 pad 2: unconnected-(SW45-Pad2) -> /R4
- SW46 pad 1: unconnected-(SW46-Pad1) -> Net-(D34-K)
- SW46 pad 2: unconnected-(SW46-Pad2) -> /R4
- SW47 pad 1: unconnected-(SW47-Pad1) -> Net-(D35-K)
- SW47 pad 2: unconnected-(SW47-Pad2) -> /R4
- SW48 pad 1: unconnected-(SW48-Pad1) -> Net-(D36-K)
- SW48 pad 2: unconnected-(SW48-Pad2) -> /R4
- SW49 pad 1: unconnected-(SW49-Pad1) -> Net-(D37-K)
- SW49 pad 2: unconnected-(SW49-Pad2) -> /R5
- SW5 pad 1: unconnected-(SW5-Pad1) -> Net-(D5-A)
- SW5 pad 2: unconnected-(SW5-Pad2) -> /R1
- SW50 pad 1: unconnected-(SW50-Pad1) -> Net-(D38-K)
- SW50 pad 2: unconnected-(SW50-Pad2) -> /R5
- SW51 pad 1: unconnected-(SW51-Pad1) -> Net-(D39-K)
- SW51 pad 2: unconnected-(SW51-Pad2) -> /R5
- SW52 pad 1: unconnected-(SW52-Pad1) -> Net-(D40-K)
- SW52 pad 2: unconnected-(SW52-Pad2) -> /R5
- SW53 pad 1: unconnected-(SW53-Pad1) -> Net-(D41-K)
- SW53 pad 2: unconnected-(SW53-Pad2) -> /R5
- SW54 pad 1: unconnected-(SW54-Pad1) -> Net-(D42-K)
- SW54 pad 2: unconnected-(SW54-Pad2) -> /R5
- SW55 pad 1: unconnected-(SW55-Pad1) -> Net-(D43-K)
- SW55 pad 2: unconnected-(SW55-Pad2) -> /R5
- SW56 pad 1: unconnected-(SW56-Pad1) -> Net-(D44-K)
- SW56 pad 2: unconnected-(SW56-Pad2) -> /R5
- SW57 pad 1: unconnected-(SW57-Pad1) -> Net-(D45-K)
- SW57 pad 2: unconnected-(SW57-Pad2) -> /R5
- SW58 pad 1: unconnected-(SW58-Pad1) -> Net-(D46-K)
- SW58 pad 2: unconnected-(SW58-Pad2) -> /R5
- SW59 pad 1: unconnected-(SW59-Pad1) -> Net-(D47-K)
- SW59 pad 2: unconnected-(SW59-Pad2) -> /R5
- SW6 pad 1: unconnected-(SW6-Pad1) -> Net-(D6-A)
- SW6 pad 2: unconnected-(SW6-Pad2) -> /R1
- SW60 pad 1: unconnected-(SW60-Pad1) -> Net-(D48-K)
- SW60 pad 2: unconnected-(SW60-Pad2) -> /R5
- SW61 pad 1: unconnected-(SW61-Pad1) -> Net-(D49-K)
- SW61 pad 2: unconnected-(SW61-Pad2) -> /R6
- SW62 pad 1: unconnected-(SW62-Pad1) -> Net-(D50-K)
- SW62 pad 2: unconnected-(SW62-Pad2) -> /R6
- SW63 pad 1: unconnected-(SW63-Pad1) -> Net-(D51-K)
- SW63 pad 2: unconnected-(SW63-Pad2) -> /R6
- SW64 pad 1: unconnected-(SW64-Pad1) -> Net-(D52-K)
- SW64 pad 2: unconnected-(SW64-Pad2) -> /R6
- SW65 pad 1: unconnected-(SW65-Pad1) -> Net-(D53-K)
- SW65 pad 2: unconnected-(SW65-Pad2) -> /R6
- SW66 pad 1: unconnected-(SW66-Pad1) -> Net-(D54-K)
- SW66 pad 2: unconnected-(SW66-Pad2) -> /R6
- SW67 pad 1: unconnected-(SW67-Pad1) -> Net-(D55-K)
- SW67 pad 2: unconnected-(SW67-Pad2) -> /R6
- SW68 pad 1: unconnected-(SW68-Pad1) -> Net-(D56-K)
- SW68 pad 2: unconnected-(SW68-Pad2) -> /R6
- SW69 pad 1: unconnected-(SW69-Pad1) -> Net-(D57-K)
- SW69 pad 2: unconnected-(SW69-Pad2) -> /R6
- SW7 pad 1: unconnected-(SW7-Pad1) -> Net-(D7-A)
- SW7 pad 2: unconnected-(SW7-Pad2) -> /R1
- SW70 pad 1: unconnected-(SW70-Pad1) -> Net-(D58-K)
- SW70 pad 2: unconnected-(SW70-Pad2) -> /R6
- SW71 pad 1: unconnected-(SW71-Pad1) -> Net-(D59-K)
- SW71 pad 2: unconnected-(SW71-Pad2) -> /R6
- SW72 pad 1: unconnected-(SW72-Pad1) -> Net-(D60-K)
- SW72 pad 2: unconnected-(SW72-Pad2) -> /R6
- SW73 pad 1: unconnected-(SW73-Pad1) -> Net-(D61-K)
- SW73 pad 2: unconnected-(SW73-Pad2) -> /R7
- SW74 pad 1: unconnected-(SW74-Pad1) -> Net-(D62-K)
- SW74 pad 2: unconnected-(SW74-Pad2) -> /R7
- SW75 pad 1: unconnected-(SW75-Pad1) -> Net-(D63-K)
- SW75 pad 2: unconnected-(SW75-Pad2) -> /R7
- SW76 pad 1: unconnected-(SW76-Pad1) -> Net-(D64-K)
- SW76 pad 2: unconnected-(SW76-Pad2) -> /R7
- SW77 pad 1: unconnected-(SW77-Pad1) -> Net-(D65-K)
- SW77 pad 2: unconnected-(SW77-Pad2) -> /R7
- SW78 pad 1: unconnected-(SW78-Pad1) -> Net-(D66-K)
- SW78 pad 2: unconnected-(SW78-Pad2) -> /R7
- SW79 pad 1: unconnected-(SW79-Pad1) -> Net-(D67-K)
- SW79 pad 2: unconnected-(SW79-Pad2) -> /R7
- SW8 pad 1: unconnected-(SW8-Pad1) -> Net-(D8-A)
- SW8 pad 2: unconnected-(SW8-Pad2) -> /R1
- SW80 pad 1: unconnected-(SW80-Pad1) -> Net-(D68-K)
- SW80 pad 2: unconnected-(SW80-Pad2) -> /R7
- SW81 pad 1: unconnected-(SW81-Pad1) -> Net-(D69-K)
- SW81 pad 2: unconnected-(SW81-Pad2) -> /R7
- SW82 pad 1: unconnected-(SW82-Pad1) -> Net-(D70-K)
- SW82 pad 2: unconnected-(SW82-Pad2) -> /R7
- SW83 pad 1: unconnected-(SW83-Pad1) -> Net-(D71-K)
- SW83 pad 2: unconnected-(SW83-Pad2) -> /R7
- SW84 pad 1: unconnected-(SW84-Pad1) -> Net-(D72-K)
- SW84 pad 2: unconnected-(SW84-Pad2) -> /R7
- SW9 pad 1: unconnected-(SW9-Pad1) -> Net-(D9-A)
- SW9 pad 2: unconnected-(SW9-Pad2) -> /R1
Routing:
- net +5V: track 0.00 -> 1869.4 mm
- net Net-(USB1-CC2): track 0.00 -> 6.05 mm
Other:
- copper layers 2 -> 4

Commit message: done
Parts:
- added J1: Testpoint, Connector_PinSocket_2.00mm:PinSocket_1x02_P2.00mm_Vertical, F.Cu at (1893.5, 637.0)
- added R3: 10k, Resistor_SMD:R_0603_1608Metric, F.Cu at (1896.7, 632.8)
- added R4: 220 ohm, Resistor_SMD:R_0603_1608Metric, F.Cu at (1811.2, 530.1)
- R1, R2, U2: moved to F.Cu
- moved R1 668.4 mm to (1970.5, 646.5), turned to 0 degrees
- moved R2 664.9 mm to (1967.4, 646.5), turned to 0 degrees
- moved USB1 659.2 mm to (1969.1, 645.5)
- moved L16 657.2 mm to (2113.4, 536.0)
- moved L31 657.2 mm to (2113.4, 555.0)
- moved L44 657.2 mm to (2065.8, 574.1)
- moved L45 657.2 mm to (2089.6, 574.1)
- moved L46 657.2 mm to (2113.4, 574.1)
- moved L60 657.2 mm to (2113.4, 593.1)
- moved L74 657.2 mm to (2113.4, 612.2)
- moved L84 657.2 mm to (2113.4, 631.2)
- moved SW16 657.2 mm to (2106.4, 533.0)
- moved SW31 657.2 mm to (2106.4, 552.0)
- moved SW44 657.2 mm to (2058.8, 571.1)
- moved SW45 657.2 mm to (2082.6, 571.1)
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Connections:
- U1 pad 1: Net-(U1-GND-Pad1) -> GND
- U1 pad 10: unconnected-(U1-IO6-Pad10) -> /C5
- U1 pad 11: unconnected-(U1-IO7-Pad11) -> /C6
- U1 pad 12: unconnected-(U1-IO8-Pad12) -> /C7
- U1 pad 13: unconnected-(U1-IO9-Pad13) -> /C8
- U1 pad 14: unconnected-(U1-IO10-Pad14) -> /C9
- U1 pad 15: unconnected-(U1-IO11-Pad15) -> /C10
- U1 pad 16: unconnected-(U1-IO12-Pad16) -> /C11
- U1 pad 17: unconnected-(U1-IO13-Pad17) -> /C12
- U1 pad 18: unconnected-(U1-IO14-Pad18) -> /R1
- U1 pad 19: unconnected-(U1-IO15-Pad19) -> /R2
- U1 pad 2: Net-(U1-GND-Pad1) -> GND
- U1 pad 20: unconnected-(U1-IO16-Pad20) -> /R3
- U1 pad 21: unconnected-(U1-IO17-Pad21) -> /R4
- U1 pad 22: unconnected-(U1-IO18-Pad22) -> /R5
- U1 pad 25: unconnected-(U1-IO21-Pad25) -> /R6
- U1 pad 30: unconnected-(U1-IO48-Pad30) -> /R7
- U1 pad 38: unconnected-(U1-IO42-Pad38) -> /GPIO42
- U1 pad 4: unconnected-(U1-IO0-Pad4) -> Net-(J1-Pin_1)
- U1 pad 42: Net-(U1-GND-Pad1) -> GND
- U1 pad 43: Net-(U1-GND-Pad1) -> GND
- U1 pad 46: Net-(U1-GND-Pad1) -> GND
- U1 pad 47: Net-(U1-GND-Pad1) -> GND
- U1 pad 48: Net-(U1-GND-Pad1) -> GND
- U1 pad 49: Net-(U1-GND-Pad1) -> GND
- U1 pad 5: unconnected-(U1-IO1-Pad5) -> /C1
- U1 pad 50: Net-(U1-GND-Pad1) -> GND
- U1 pad 51: Net-(U1-GND-Pad1) -> GND
- U1 pad 52: Net-(U1-GND-Pad1) -> GND
- U1 pad 53: Net-(U1-GND-Pad1) -> GND
- U1 pad 54: Net-(U1-GND-Pad1) -> GND
- U1 pad 55: Net-(U1-GND-Pad1) -> GND
- U1 pad 56: Net-(U1-GND-Pad1) -> GND
- U1 pad 57: Net-(U1-GND-Pad1) -> GND
- U1 pad 58: Net-(U1-GND-Pad1) -> GND
- U1 pad 59: Net-(U1-GND-Pad1) -> GND
- U1 pad 6: unconnected-(U1-IO2-Pad6) -> /C2
- U1 pad 60: Net-(U1-GND-Pad1) -> GND
- U1 pad 61: Net-(U1-GND-Pad1) -> GND
- U1 pad 62: Net-(U1-GND-Pad1) -> GND
- U1 pad 63: Net-(U1-GND-Pad1) -> GND
- U1 pad 64: Net-(U1-GND-Pad1) -> GND
- U1 pad 65: Net-(U1-GND-Pad1) -> GND
- U1 pad 8: unconnected-(U1-IO4-Pad8) -> /C3
- U1 pad 9: unconnected-(U1-IO5-Pad9) -> /C4
- U2 pad 2: /GPIO -> /GPIO42
- U2 pad 4: /DIN -> Net-(R4-Pad1)
Routing:
- net /R2: track 0.00 -> 668.7 mm
- net +5V: track 1869.4 -> 2321.2 mm, vias 0 -> 90
- net /R1: track 0.00 -> 398.1 mm
- net /R4: track 0.00 -> 373.5 mm, vias 0 -> 5
- net /R3: track 0.00 -> 355.2 mm, vias 0 -> 8
- net /R7: track 0.00 -> 327.1 mm, vias 0 -> 2
- net Net-(L16-DOUT): track 0.00 -> 316.8 mm, vias 0 -> 3
- net /R5: track 0.00 -> 303.8 mm, vias 0 -> 3
- net Net-(L31-DOUT): track 0.00 -> 303.6 mm, vias 0 -> 2
- net Net-(L74-DOUT): track 0.00 -> 299.7 mm
- net Net-(L46-DOUT): track 0.00 -> 288.6 mm, vias 0 -> 2
- net /EOS5: track 0.00 -> 283.5 mm
- net Net-(D48-K): track 0.00 -> 269.9 mm, vias 0 -> 2
- net Net-(D18-K): track 0.00 -> 264.8 mm, vias 0 -> 1
- net Net-(D61-K): track 0.00 -> 264.6 mm
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- added copper zone on In2.Cu, net GND
Other:
- board outline added: 311.2 x 123 mm
- board text added: "Testpoint"

Commit message: done 3d model finding
Parts:
- SW1, SW10, SW11, SW12, SW13, SW14, SW15, SW16, SW17, SW18, SW19, SW2, SW20, SW21, SW22, SW23, SW24, SW25, SW26, SW27, SW28, SW29, SW3, SW30, SW31, SW32, SW33, SW34, SW35, SW36, SW37, SW38, SW39, SW4, SW40, SW41, SW42, SW43, SW44, SW45, SW46, SW47, SW48, SW49, SW5, SW50, SW51, SW52, SW53, SW54, SW55, SW56, SW57, SW58, SW59, SW6, SW60, SW61, SW62, SW63, SW64, SW65, SW66, SW67, SW68, SW69, SW7, SW70, SW71, SW72, SW73, SW74, SW75, SW76, SW77, SW78, SW79, SW8, SW80, SW81, SW82, SW83, SW84, SW9: footprint Button_Switch_Keyboard:SW_Cherry_MX_1.00u_PCB -> Library:switch

Commit message: made vias bigger and added ams
Parts:
- added U3: AMS1117, Package_TO_SOT_SMD:SOT-223-3_TabPin2, B.Cu at (1890.7, 625.6)
- SW1, SW10, SW11, SW12, SW13, SW14, SW15, SW16, SW17, SW18, SW19, SW2, SW20, SW21, SW22, SW23, SW24, SW25, SW26, SW27, SW28, SW29, SW3, SW30, SW31, SW32, SW33, SW34, SW35, SW36, SW37, SW38, SW39, SW4, SW40, SW41, SW42, SW43, SW44, SW45, SW46, SW47, SW48, SW49, SW5, SW50, SW51, SW52, SW53, SW54, SW55, SW56, SW57, SW58, SW59, SW6, SW60, SW61, SW62, SW63, SW64, SW65, SW66, SW67, SW68, SW69, SW7, SW70, SW71, SW72, SW73, SW74, SW75, SW76, SW77, SW78, SW79, SW8, SW80, SW81, SW82, SW83, SW84, SW9: footprint Library:switch -> Button_Switch_Keyboard:SW_Cherry_MX_1.00u_PCB
Connections:
- U1 pad 3: unconnected-(U1-3V3-Pad3) -> /3.3v
Routing:
- net /3.3v: track 0.00 -> 32.4 mm, vias 0 -> 4
- net +5V: track 2321.2 -> 2336.5 mm, vias 90 -> 91
- net GND: track 165.7 -> 167.9 mm, vias 98 -> 99
